Commit message: 更新 Taks T1 机器人 URDF/XML 配置和网格文件
修正机器人模型的惯性参数、关节原点和速度限制:
- 调整 pelvis、waist_roll_link、torso_link 等连杆的惯性矩阵
- 修正左右髋关节和腰部偏航关节的原点位置和旋转角度
- 更新踝关节、肩关节、肘关节和腕关节的速度限制值
- 更新 pelvis 和 left_hip_yaw_link 网格文件
- 删除未使用的 base_link.STL 网格文件
- 添加重定向和录制命令的使用说明

File: assets/Taks_T1/Taks_T1.urdf (robot description, URDF)
Before this commit: robot Taks_T1, 33 links, 32 joints
Joints:
- joint left_ankle_pitch_joint: limit lower=-0.87267 upper=0.5236 effort=27.0 velocity=3.77 -> lower=-0.87267 upper=0.5236 effort=27.0 velocity=5.4454
- joint left_ankle_roll_joint: limit lower=-0.2618 upper=0.2618 effort=27.0 velocity=3.77 -> lower=-0.2618 upper=0.2618 effort=27.0 velocity=5.4454
- joint left_elbow_joint: limit lower=-0.7 upper=1.57 effort=27.0 velocity=3.77 -> lower=-0.7 upper=1.57 effort=27.0 velocity=5.4454
- joint left_hip_pitch_joint: origin xyz=0.115 0.0 -0.0523 rpy=0.0 0.0 -1.5707963267948966 -> xyz=0.0 0.115 -0.0523 rpy=0 0 0
- joint left_shoulder_pitch_joint: limit lower=-3.0 upper=2.0 effort=27.0 velocity=3.77 -> lower=-3.0 upper=2.0 effort=27.0 velocity=5.4454
- joint left_shoulder_roll_joint: limit lower=-0.2 upper=2.2515 effort=27.0 velocity=3.77 -> lower=-0.2 upper=2.2515 effort=27.0 velocity=5.4454
- joint left_shoulder_yaw_joint: limit lower=-2.58 upper=2.58 effort=27.0 velocity=3.77 -> lower=-2.58 upper=2.58 effort=27.0 velocity=5.4454
- joint left_wrist_pitch_joint: limit lower=-0.9 upper=0.9 effort=7.0 velocity=12.57 -> lower=-0.9 upper=0.9 effort=7.0 velocity=20.944
- joint left_wrist_roll_joint: limit lower=-2.67 upper=2.67 effort=7.0 velocity=12.57 -> lower=-2.67 upper=2.67 effort=7.0 velocity=20.944
- joint left_wrist_yaw_joint: limit lower=-0.9 upper=0.9 effort=7.0 velocity=12.57 -> lower=-0.9 upper=0.9 effort=7.0 velocity=20.944
- joint right_ankle_pitch_joint: limit lower=-0.87267 upper=0.5236 effort=27.0 velocity=3.77 -> lower=-0.87267 upper=0.5236 effort=27.0 velocity=5.4454
- joint right_ankle_roll_joint: limit lower=-0.2618 upper=0.2618 effort=27.0 velocity=3.77 -> lower=-0.2618 upper=0.2618 effort=27.0 velocity=5.4454
- joint right_elbow_joint: limit lower=-0.7 upper=1.57 effort=27.0 velocity=3.77 -> lower=-0.7 upper=1.57 effort=27.0 velocity=5.4454
- joint right_hip_pitch_joint: origin xyz=-0.115 0.0 -0.0523 rpy=0.0 0.0 -1.5707963267948966 -> xyz=0.0 -0.115 -0.0523 rpy=0 0 0
- joint right_shoulder_pitch_joint: limit lower=-2.0 upper=2.0 effort=27.0 velocity=3.77 -> lower=-2.0 upper=2.0 effort=27.0 velocity=5.4454
- joint right_shoulder_roll_joint: limit lower=-2.2515 upper=0.2 effort=27.0 velocity=3.77 -> lower=-2.2515 upper=0.2 effort=27.0 velocity=5.4454
- joint right_shoulder_yaw_joint: limit lower=-2.58 upper=2.58 effort=27.0 velocity=3.77 -> lower=-2.58 upper=2.58 effort=27.0 velocity=5.4454
- joint right_wrist_pitch_joint: limit lower=-0.9 upper=0.9 effort=7.0 velocity=12.57 -> lower=-0.9 upper=0.9 effort=7.0 velocity=20.944
- joint right_wrist_roll_joint: limit lower=-2.67 upper=2.67 effort=7.0 velocity=12.57 -> lower=-2.67 upper=2.67 effort=7.0 velocity=20.944
- joint right_wrist_yaw_joint: limit lower=-0.9 upper=0.9 effort=7.0 velocity=12.57 -> lower=-0.9 upper=0.9 effort=7.0 velocity=20.944
- joint waist_yaw_joint: origin xyz=0.0 0.0 0.0 rpy=0.0 0.0 -1.5707963267948966 -> xyz=0.0 0.0 0.0 rpy=0 0 0

Commit message: 优化 Taks T1 机器人碰撞检测配置和人体尺度参数
- 在 URDF 中为左右踝关节连杆添加碰撞几何体(使用 STL 网格)
- 在 XML 中为所有碰撞几何体统一添加 contype="1" conaffinity="1" 属性以启用碰撞检测
- 添加完整的场景配置,包括天空盒、地面纹理、材质定义和定向光源
- 在 contact 标签中添加 36 对相邻关节的碰撞排除规则,避免自碰撞
- 调整 BVH LAFAN1、FBX 和 SMPLX 三种格式的人体尺度缩放参数:

File: assets/Taks_T1/Taks_T1.urdf (robot description, URDF)
Before this commit: robot Taks_T1, 33 links, 32 joints
Links:
- link left_ankle_roll_link: geometry collision mesh filename=meshes/left_ankle_roll_link.STL; visual mesh filename=meshes/left_ankle_roll_link.STL
- link right_ankle_roll_link: geometry collision mesh filename=meshes/right_ankle_roll_link.STL; visual mesh filename=meshes/right_ankle_roll_link.STL

Commit message: 更新mjcf碰撞体

File: assets/Taks_T1/Taks_T1.urdf (robot description, URDF)
Before this commit: robot Taks_T1, 33 links, 32 joints
Links:
- link left_ankle_pitch_link: geometry collision sphere radius=0.02; visual mesh filename=../meshes/left_ankle_pitch_link.STL
- link left_ankle_roll_link: geometry collision box size=0.26 0.12 0.025; visual mesh filename=../meshes/left_ankle_roll_link.STL
- link left_elbow_link: geometry collision sphere radius=0.045; visual mesh filename=../meshes/left_elbow_link.STL
- link left_hip_pitch_link: geometry collision sphere radius=0.05; visual mesh filename=../meshes/left_hip_pitch_link.STL
- link left_hip_roll_link: geometry collision sphere radius=0.055; visual mesh filename=../meshes/left_hip_roll_link.STL
- link left_hip_yaw_link: geometry collision cylinder length=0.2 radius=0.05; visual mesh filename=../meshes/left_hip_yaw_link.STL
- link left_knee_link: geometry collision cylinder length=0.24 radius=0.04; visual mesh filename=../meshes/left_knee_link.STL
- link left_shoulder_pitch_link: geometry collision sphere radius=0.04; visual mesh filename=../meshes/left_shoulder_pitch_link.STL
- link left_shoulder_roll_link: geometry collision sphere radius=0.05; visual mesh filename=../meshes/left_shoulder_roll_link.STL
- link left_shoulder_yaw_link: geometry collision cylinder length=0.14 radius=0.035; visual mesh filename=../meshes/left_shoulder_yaw_link.STL
- link left_wrist_pitch_link: geometry collision cylinder length=0.1 radius=0.025; visual mesh filename=../meshes/left_wrist_pitch_link.STL
- link left_wrist_roll_link: geometry collision cylinder length=0.1 radius=0.025; visual mesh filename=../meshes/left_wrist_roll_link.STL
- link left_wrist_yaw_link: geometry collision sphere radius=0.03; visual mesh filename=../meshes/left_wrist_yaw_link.STL
- link neck_pitch_link: geometry collision sphere radius=0.09; visual mesh filename=../meshes/neck_pitch_link.STL
- link neck_roll_link: geometry collision cylinder length=0.06 radius=0.015; visual mesh filename=../meshes/neck_roll_link.STL
- link neck_yaw_link: geometry collision cylinder length=0.06 radius=0.03; visual mesh filename=../meshes/neck_yaw_link.STL
- link pelvis: geometry collision box size=0.16 0.2 0.12; visual mesh filename=../meshes/pelvis.STL
- link right_ankle_pitch_link: geometry collision sphere radius=0.02; visual mesh filename=../meshes/right_ankle_pitch_link.STL
- link right_ankle_roll_link: geometry collision box size=0.26 0.12 0.025; visual mesh filename=../meshes/right_ankle_roll_link.STL
- link right_elbow_link: geometry collision sphere radius=0.045; visual mesh filename=../meshes/right_elbow_link.STL
- link right_hip_pitch_link: geometry collision sphere radius=0.05; visual mesh filename=../meshes/right_hip_pitch_link.STL
- link right_hip_roll_link: geometry collision sphere radius=0.055; visual mesh filename=../meshes/right_hip_roll_link.STL
- link right_hip_yaw_link: geometry collision cylinder length=0.2 radius=0.05; visual mesh filename=../meshes/right_hip_yaw_link.STL
- link right_knee_link: geometry collision cylinder length=0.24 radius=0.04; visual mesh filename=../meshes/right_knee_link.STL
- link right_shoulder_pitch_link: geometry collision sphere radius=0.04; visual mesh filename=../meshes/right_shoulder_pitch_link.STL
- link right_shoulder_roll_link: geometry collision sphere radius=0.05; visual mesh filename=../meshes/right_shoulder_roll_link.STL
- link right_shoulder_yaw_link: geometry collision cylinder length=0.14 radius=0.035; visual mesh filename=../meshes/right_shoulder_yaw_link.STL
- link right_wrist_pitch_link: geometry collision cylinder length=0.1 radius=0.025; visual mesh filename=../meshes/right_wrist_pitch_link.STL
- link right_wrist_roll_link: geometry collision cylinder length=0.1 radius=0.025; visual mesh filename=../meshes/right_wrist_roll_link.STL
- link right_wrist_yaw_link: geometry collision sphere radius=0.03; visual mesh filename=../meshes/right_wrist_yaw_link.STL
- link torso_link: geometry collision box size=0.22 0.20 0.20; visual mesh filename=../meshes/waist_pitch_link.STL
- link waist_roll_link: geometry collision cylinder length=0.06 radius=0.06; visual mesh filename=../meshes/waist_roll_link.STL
- link waist_yaw_link: geometry collision cylinder length=0.04 radius=0.06; visual mesh filename=../meshes/waist_yaw_link.STL

Commit message: 更新 Taks_T1 URDF 文件:统一碰撞体为 mesh 格式并修正文件路径
- 将所有碰撞体从简单几何形状(box、sphere、cylinder)改为使用 mesh 文件
- 统一所有碰撞体的 origin 为 xyz="0 0 0" rpy="0 0 0"
- 修正 mesh 文件路径:从 "../meshes/" 改为 "meshes/"
- 简化 mujoco 碰撞配置:移除大部分关节的 mujoco geom 标签,仅保留 pelvis、waist 和上肢关键部位
- 统一保留部位的 contype 和 conaffinity 参数为更简洁的配置

File: assets/Taks_T1/Taks_T1.urdf (robot description, URDF)
Before this commit: robot Taks_T1, 33 links, 32 joints
Links:
- link left_ankle_pitch_link: geometry collision mesh filename=meshes/left_ankle_pitch_link.STL; visual mesh filename=meshes/left_ankle_pitch_link.STL
- link left_ankle_roll_link: geometry collision mesh filename=meshes/left_ankle_roll_link.STL; visual mesh filename=meshes/left_ankle_roll_link.STL
- link left_elbow_link: geometry collision mesh filename=meshes/left_elbow_link.STL; visual mesh filename=meshes/left_elbow_link.STL
- link left_hip_pitch_link: geometry collision mesh filename=meshes/left_hip_pitch_link.STL; visual mesh filename=meshes/left_hip_pitch_link.STL
- link left_hip_roll_link: geometry collision mesh filename=meshes/left_hip_roll_link.STL; visual mesh filename=meshes/left_hip_roll_link.STL
- link left_hip_yaw_link: geometry collision mesh filename=meshes/left_hip_yaw_link.STL; visual mesh filename=meshes/left_hip_yaw_link.STL
- link left_knee_link: geometry collision mesh filename=meshes/left_knee_link.STL; visual mesh filename=meshes/left_knee_link.STL
- link left_shoulder_pitch_link: geometry collision mesh filename=meshes/left_shoulder_pitch_link.STL; visual mesh filename=meshes/left_shoulder_pitch_link.STL
- link left_shoulder_roll_link: geometry collision mesh filename=meshes/left_shoulder_roll_link.STL; visual mesh filename=meshes/left_shoulder_roll_link.STL
- link left_shoulder_yaw_link: geometry collision mesh filename=meshes/left_shoulder_yaw_link.STL; visual mesh filename=meshes/left_shoulder_yaw_link.STL
- link left_wrist_pitch_link: geometry collision mesh filename=meshes/left_wrist_pitch_link.STL; visual mesh filename=meshes/left_wrist_pitch_link.STL
- link left_wrist_roll_link: geometry collision mesh filename=meshes/left_wrist_roll_link.STL; visual mesh filename=meshes/left_wrist_roll_link.STL
- link left_wrist_yaw_link: geometry collision mesh filename=meshes/left_wrist_yaw_link.STL; visual mesh filename=meshes/left_wrist_yaw_link.STL
- link neck_pitch_link: geometry collision mesh filename=meshes/neck_pitch_link.STL; visual mesh filename=meshes/neck_pitch_link.STL
- link neck_roll_link: geometry collision mesh filename=meshes/neck_roll_link.STL; visual mesh filename=meshes/neck_roll_link.STL
- link neck_yaw_link: geometry collision mesh filename=meshes/neck_yaw_link.STL; visual mesh filename=meshes/neck_yaw_link.STL
- link pelvis: geometry collision mesh filename=meshes/pelvis.STL; visual mesh filename=meshes/pelvis.STL
- link right_ankle_pitch_link: geometry collision mesh filename=meshes/right_ankle_pitch_link.STL; visual mesh filename=meshes/right_ankle_pitch_link.STL
- link right_ankle_roll_link: geometry collision mesh filename=meshes/right_ankle_roll_link.STL; visual mesh filename=meshes/right_ankle_roll_link.STL
- link right_elbow_link: geometry collision mesh filename=meshes/right_elbow_link.STL; visual mesh filename=meshes/right_elbow_link.STL
- link right_hip_pitch_link: geometry collision mesh filename=meshes/right_hip_pitch_link.STL; visual mesh filename=meshes/right_hip_pitch_link.STL
- link right_hip_roll_link: geometry collision mesh filename=meshes/right_hip_roll_link.STL; visual mesh filename=meshes/right_hip_roll_link.STL
- link right_hip_yaw_link: geometry collision mesh filename=meshes/right_hip_yaw_link.STL; visual mesh filename=meshes/right_hip_yaw_link.STL
- link right_knee_link: geometry collision mesh filename=meshes/right_knee_link.STL; visual mesh filename=meshes/right_knee_link.STL
- link right_shoulder_pitch_link: geometry collision mesh filename=meshes/right_shoulder_pitch_link.STL; visual mesh filename=meshes/right_shoulder_pitch_link.STL
- link right_shoulder_roll_link: geometry collision mesh filename=meshes/right_shoulder_roll_link.STL; visual mesh filename=meshes/right_shoulder_roll_link.STL
- link right_shoulder_yaw_link: geometry collision mesh filename=meshes/right_shoulder_yaw_link.STL; visual mesh filename=meshes/right_shoulder_yaw_link.STL
- link right_wrist_pitch_link: geometry collision mesh filename=meshes/right_wrist_pitch_link.STL; visual mesh filename=meshes/right_wrist_pitch_link.STL
- link right_wrist_roll_link: geometry collision mesh filename=meshes/right_wrist_roll_link.STL; visual mesh filename=meshes/right_wrist_roll_link.STL
- link right_wrist_yaw_link: geometry collision mesh filename=meshes/right_wrist_yaw_link.STL; visual mesh filename=meshes/right_wrist_yaw_link.STL
- link torso_link: geometry collision mesh filename=meshes/waist_pitch_link.STL; visual mesh filename=meshes/waist_pitch_link.STL
- link waist_roll_link: geometry collision mesh filename=meshes/waist_roll_link.STL; visual mesh filename=meshes/waist_roll_link.STL
- link waist_yaw_link: geometry collision mesh filename=meshes/waist_yaw_link.STL; visual mesh filename=meshes/waist_yaw_link.STL
