Commit message: 更新Semi_Taks_LV1机器人模型的惯性参数和关节配置
- 移除URDF编译器中的balanceinertia选项
- 重新计算所有link的惯性参数（质量、质心位置、惯性张量）
- 调整关节原点位置和限位角度
- 统一更新所有关节的armature动力学参数
- 交换waist_pitch和waist_roll关节的父子关系
- 为waist_roll_link添加多个视觉和碰撞网格组件
- 添加right_arm_long_link_active_aux辅助连杆及关节
- 微调肩部、肘部、腕部关节的位

File: assets/Semi_Taks_LV1/Semi_Taks_LV1.urdf (robot description, URDF)
Before this commit: robot Semi_Taks_LV1, 46 links, 45 joints
Links:
- removed link head_front_link_active_link
- removed link head_front_link_bevel_gear_link
- removed link head_front_link_motor_link
- removed link head_rear_link_active_link
- removed link head_rear_link_bevel_gear_link
- removed link head_rear_link_motor_link
- added link left_arm_long_link_active_aux_link, mass 0.00932618985795366; collision mesh filename=meshes/left_arm_long_link_active_aux_link.STL; visual mesh filename=meshes/left_arm_long_link_active_aux_link.STL
- added link left_arm_short_link_active_aux_link, mass 0.005963591608481944; collision mesh filename=meshes/left_arm_short_link_active_aux_link.STL; visual mesh filename=meshes/left_arm_short_link_active_aux_link.STL
- added link right_arm_long_link_active_aux_link, mass 0.00932618985795366; collision mesh filename=meshes/right_arm_long_link_active_aux_link.STL; visual mesh filename=meshes/right_arm_long_link_active_aux_link.STL
- added link right_arm_short_link_active_aux_link, mass 0.005963591608481943; collision mesh filename=meshes/right_arm_short_link_active_aux_link.STL; visual mesh filename=meshes/right_arm_short_link_active_aux_link.STL
- link base_link: mass 2.0612 -> 2.018963361217213
- link head_pitch_link: mass 0.0570635 -> 0.03003272441544096
- link head_roll_link: mass 0.0979261 -> 0.009803523609653924
- link head_yaw_link: mass 0.890304 -> 0.3247772520646972
- link left_arm_long_link_active_link: mass 0.0122523 -> 0.009326189857953662
- link left_arm_long_link_bevel_gear_link: mass 0.0416771 -> 0.01251816161658807
- link left_arm_long_link_motor_link: mass 0.00963967 -> 0.007282671248581928
- link left_arm_short_link_active_link: mass 0.00666865 -> 0.005963591608481943
- link left_arm_short_link_bevel_gear_link: mass 0.0416771 -> 0.01251816161658807
- link left_arm_short_link_motor_link: mass 0.00963967 -> 0.007282671248581928
- link left_elbow_link: mass 1.01213 -> 0.2896934028131387
- link left_shoulder_pitch_link: mass 0.74762 -> 0.5580897239034346
- link left_shoulder_roll_link: mass 1.02418 -> 0.5515329270413285
- link left_shoulder_yaw_link: mass 0.826006 -> 0.5566379737825708
- link left_wrist_pitch_link: mass 0.141783 -> 0.3726023090550386
- link left_wrist_roll_link: mass 0.797562 -> 0.5136894537866243
- link left_wrist_yaw_link: mass 0.098024 -> 0.009803523609653926
- link right_arm_long_link_active_link: mass 0.0122523 -> 0.00932618985795366
- link right_arm_long_link_bevel_gear_link: mass 0.0416771 -> 0.01251816161658807
- link right_arm_long_link_motor_link: mass 0.00963967 -> 0.007282671248581928
- link right_arm_short_link_active_link: mass 0.00666865 -> 0.005963591608481944
- link right_arm_short_link_bevel_gear_link: mass 0.0416771 -> 0.01251816161658807
- link right_arm_short_link_motor_link: mass 0.00963967 -> 0.007282671248581928
- link right_elbow_link: mass 1.01213 -> 0.2896934028131386
- link right_shoulder_pitch_link: mass 0.74762 -> 0.5580897239034346
- link right_shoulder_roll_link: mass 1.02418 -> 0.5515329270413285
- link right_shoulder_yaw_link: mass 0.826006 -> 0.5566379737825702
- link right_wrist_pitch_link: mass 0.141783 -> 0.3726023090915405
- link right_wrist_roll_link: mass 0.797562 -> 0.5136894537866242
- link right_wrist_yaw_link: mass 0.098024 -> 0.009803523609653924
- link waist_left_link_driven_link: mass 0.0123329 -> 0.01206529948233483
- link waist_left_motor_link: mass 0.556801 -> 0.06153448822481092
- link waist_pitch_link: mass 4.95555 -> 0.05005758358315827
- link waist_right_link_driven_link: mass 0.0123329 -> 0.01206529948233483
- link waist_right_motor_link: mass 0.556801 -> 0.06153448822481092
- link waist_roll_link: mass 0.145538 -> 3.941099362092086; geometry collision mesh filename=meshes/waist_roll_link.STL; collision mesh filename=meshes/waist_roll_link_left_shoulder_mount.STL
- link waist_yaw_link: mass 0.353551 -> 0.1232393527960049
Joints:
- removed joint head_front_link_active_joint
- removed joint head_front_link_bevel_gear_joint
- removed joint head_front_link_motor_joint
- removed joint head_rear_link_active_joint
- removed joint head_rear_link_bevel_gear_joint
- removed joint head_rear_link_motor_joint
- added joint left_arm_long_link_active_aux_joint: type revolute, parent left_arm_long_link_motor_link, child left_arm_long_link_active_aux_link, origin xyz=0 -0.012 0 rpy=0 0 0, axis 0 0 1, limit lower=-3.1415 upper=3.1415 effort=0 velocity=0
- added joint left_arm_short_link_active_aux_joint: type revolute, parent left_arm_short_link_motor_link, child left_arm_short_link_active_aux_link, origin xyz=0 0.012 0 rpy=0 0 0, axis 0 0 1, limit lower=-3.1415 upper=3.1415 effort=0 velocity=0
- added joint right_arm_long_link_active_aux_joint: type revolute, parent right_arm_long_link_motor_link, child right_arm_long_link_active_aux_link, origin xyz=0 0.012 0 rpy=0 0 0, axis 0 0 1, limit lower=-3.1415 upper=3.1415 effort=0 velocity=0
- added joint right_arm_short_link_active_aux_joint: type revolute, parent right_arm_short_link_motor_link, child right_arm_short_link_active_aux_link, origin xyz=0 -0.012 0 rpy=0 0 0, axis 0 0 1, limit lower=-3.1415 upper=3.1415 effort=0 velocity=0
- joint head_left_camera_joint: origin xyz=0.08538 0.02451 0.05648 rpy=0 0.17453 0 -> xyz=0.08812307593 0.02999965544 0.05311159739 rpy=0 0.172787596 0
- joint head_right_camera_joint: origin xyz=0.08538 -0.02347 0.05648 rpy=0 0.17453 0 -> xyz=0.08812307593 -0.03000034456 0.05311159739 rpy=0 0.172787596 0
- joint head_roll_joint: limit lower=-3.1415 upper=3.1415 effort=0 velocity=0 -> lower=-1.5708 upper=1.5708 effort=6 velocity=12.57; origin xyz=-0.0044 0 0.42 rpy=0 0 0 -> xyz=-0.0047 -0.0002 0.4075 rpy=0 0 0; parent waist_pitch_link -> waist_roll_link
- joint head_yaw_joint: origin xyz=0 0 0.03589 rpy=0 0 0 -> xyz=0 0 0.04 rpy=0 0 0
- joint left_arm_long_link_active_joint: origin xyz=0 0.012 0.005 rpy=0 0 0 -> xyz=0 0.012 0 rpy=0 0 0
- joint left_arm_long_link_bevel_gear_joint: origin xyz=0 0 0.01053 rpy=0 0 0 -> xyz=0 0 0.0267 rpy=0 0 0
- joint left_arm_long_link_motor_joint: limit lower=-0.9885 upper=0.9885 effort=6 velocity=12.57 -> lower=-1.2217 upper=1.2217 effort=6 velocity=12.57; origin xyz=0.026 0 0.0262 rpy=0 0 0 -> xyz=0.026 0 0.0267 rpy=0 0 0
- joint left_arm_short_link_active_joint: origin xyz=0 -0.012 -0.005 rpy=0 0 0 -> xyz=0 -0.012 0 rpy=0 0 0
- joint left_arm_short_link_bevel_gear_joint: origin xyz=0 0 -0.01053 rpy=0 0 0 -> xyz=0 0 -0.0263 rpy=0 0 0
- joint left_arm_short_link_motor_joint: limit lower=-0.9885 upper=0.9885 effort=6 velocity=12.57 -> lower=-1.2217 upper=1.2217 effort=6 velocity=12.57; origin xyz=0.073 0 -0.0262 rpy=0 0 0 -> xyz=0.073 0 -0.0263 rpy=0 0 0
- joint left_elbow_joint: limit lower=-1.0472 upper=1.35 effort=30 velocity=3.77 -> lower=-1.0472 upper=1.5708 effort=30 velocity=3.77; origin xyz=0.003 0.030399 -0.058695 rpy=0 0 0 -> xyz=0.003 0.0356 -0.0552 rpy=0 0 0
- joint left_shoulder_pitch_joint: origin xyz=-0.0048 0.097855 0.316745 rpy=0 0 0 -> xyz=-0.0048 0.097855 0.310745 rpy=0 0 0; parent waist_pitch_link -> waist_roll_link
- joint left_shoulder_roll_joint: origin xyz=0.0325 0.049045 -0.021665 rpy=0 0 0 -> xyz=0.042 0.049045 -0.021645 rpy=0 0 0
- joint left_shoulder_yaw_joint: origin xyz=-0.0275 0.015 -0.161305 rpy=0 0 0 -> xyz=-0.0378 0.015 -0.16582 rpy=0 0 0
- joint left_wrist_pitch_joint: limit lower=-1.57 upper=1.57 effort=6 velocity=12.57 -> lower=-1.5708 upper=1.5708 effort=6 velocity=12.57
- joint left_wrist_roll_joint: origin xyz=0.09743 -0.030399 -0.025 rpy=0 0 0 -> xyz=0.0972 -0.0305 -0.025 rpy=0 0 0
- joint left_wrist_yaw_joint: limit lower=-3.1415 upper=3.1415 effort=0 velocity=0 -> lower=-1.5708 upper=1.5708 effort=6 velocity=12.57; origin xyz=0.127 0 0 rpy=0 0 0 -> xyz=0.1255 0 0 rpy=0 0 0
- joint right_arm_long_link_active_joint: origin xyz=0 -0.012 0.005 rpy=0 0 0 -> xyz=0 -0.012 0 rpy=0 0 0
- joint right_arm_long_link_bevel_gear_joint: origin xyz=0 0 0.01053 rpy=0 0 0 -> xyz=0 0 0.0267 rpy=0 0 0
- joint right_arm_long_link_motor_joint: limit lower=-0.9885 upper=0.9885 effort=6 velocity=12.57 -> lower=-1.2217 upper=1.2217 effort=6 velocity=12.57; origin xyz=0.026 0 0.0262 rpy=0 0 0 -> xyz=0.026 0 0.0267 rpy=0 0 0
- joint right_arm_short_link_active_joint: origin xyz=0 0.012 -0.005 rpy=0 0 0 -> xyz=0 0.012 0 rpy=0 0 0
- joint right_arm_short_link_bevel_gear_joint: origin xyz=0 0 -0.01053 rpy=0 0 0 -> xyz=0 0 -0.0263 rpy=0 0 0
- joint right_arm_short_link_motor_joint: limit lower=-0.9885 upper=0.9885 effort=6 velocity=12.57 -> lower=-1.2217 upper=1.2217 effort=6 velocity=12.57; origin xyz=0.073 0 -0.0262 rpy=0 0 0 -> xyz=0.073 0 -0.0263 rpy=0 0 0
- joint right_elbow_joint: limit lower=-1.0472 upper=1.35 effort=30 velocity=3.77 -> lower=-1.0472 upper=1.5708 effort=30 velocity=3.77; origin xyz=0.003 -0.030399 -0.058695 rpy=0 0 0 -> xyz=0.003 -0.0356 -0.0552 rpy=0 0 0
- joint right_shoulder_pitch_joint: origin xyz=-0.0048 -0.097855 0.316745 rpy=0 0 0 -> xyz=-0.0048 -0.097855 0.310745 rpy=0 0 0; parent waist_pitch_link -> waist_roll_link
- joint right_shoulder_roll_joint: origin xyz=0.0325 -0.049045 -0.021665 rpy=0 0 0 -> xyz=0.042 -0.049045 -0.021645 rpy=0 0 0
- joint right_shoulder_yaw_joint: origin xyz=-0.0275 -0.015 -0.161305 rpy=0 0 0 -> xyz=-0.0378 -0.015 -0.16582 rpy=0 0 0
- joint right_wrist_pitch_joint: limit lower=-1.57 upper=1.57 effort=6 velocity=12.57 -> lower=-1.5708 upper=1.5708 effort=6 velocity=12.57
- joint right_wrist_roll_joint: origin xyz=0.09743 0.030399 -0.025 rpy=0 0 0 -> xyz=0.0972 0.0305 -0.025 rpy=0 0 0
- joint right_wrist_yaw_joint: limit lower=-3.1415 upper=3.1415 effort=0 velocity=0 -> lower=-1.5708 upper=1.5708 effort=6 velocity=12.57; origin xyz=0.127 0 0 rpy=0 0 0 -> xyz=0.1255 0 0 rpy=0 0 0
- joint waist_left_link_driven_joint: origin xyz=0.0341 0.022 0.0195 rpy=0 0 0 -> xyz=0.03415 0.022 0.0195 rpy=0 0 0
- joint waist_left_motor_joint: limit lower=-1.0908 upper=1.0908 effort=60 velocity=4.19 -> lower=-1.16190000 upper=0.75000000 effort=60 velocity=4.19; origin xyz=0.02085 0.0425 0.052 rpy=0 0 0 -> xyz=0.02515 0.0425 0.052 rpy=0 0 0; parent waist_pitch_link -> waist_roll_link
- joint waist_pitch_joint: origin xyz=0 0 0 rpy=0 0 0 -> xyz=0 0 0.0355 rpy=0 0 0; parent waist_roll_link -> waist_yaw_link
- joint waist_right_link_driven_joint: origin xyz=0.0341 -0.022 0.0195 rpy=0 0 0 -> xyz=0.03415 -0.0221 0.0195 rpy=0 0 0
- joint waist_right_motor_joint: limit lower=-1.0908 upper=1.0908 effort=60 velocity=4.19 -> lower=-0.75000000 upper=1.16190000 effort=60 velocity=4.19; origin xyz=0.02085 -0.0425 0.052 rpy=0 0 0 -> xyz=0.02515 -0.0425 0.052 rpy=0 0 0; parent waist_pitch_link -> waist_roll_link
- joint waist_roll_joint: origin xyz=0 0 0.0355 rpy=0 0 0 -> xyz=0 0 0 rpy=0 0 0; parent waist_yaw_link -> waist_pitch_link
- joint waist_yaw_joint: origin xyz=0 0 0.0638 rpy=0 0 0 -> xyz=0 0 0.0698 rpy=0 0 0

Commit message: [update] Semi_Taks_LV1 neck motor parameters and fixed-base retargeting improvements
- Increase neck joint effort limits from 3 to 12.5 N⋅m
- Reduce neck joint velocity limits by ~50% for safer operation
- Increase neck motor armature from 0.000426 to 0.0019
- Update neck PD gains to match wrist motors (kp=7.5, kv=0.48)
- Add fixed_base_heading_offset parameter to IK configs
- Implement FixedBaseTargets class for proper fixed-base retargeting
- Fix robot root position calculation to use configuration

File: assets/Semi_Taks_LV1/Semi_Taks_LV1.urdf (robot description, URDF)
Before this commit: robot Semi_Taks_LV1, 25 links, 24 joints
Joints:
- joint head_pitch_joint: limit lower=-1.57 upper=1.57 effort=3 velocity=95.29497715889039 -> lower=-1.57 upper=1.57 effort=12.5 velocity=47.12388980384689
- joint head_yaw_joint: limit lower=-2.618 upper=2.618 effort=3 velocity=95.29497715889039 -> lower=-2.618 upper=2.618 effort=12.5 velocity=47.12388980384689
